File: design/ACS_PCB.kicad_sch (KiCad schematic)
At the start: 32 parts, among them J1 USB_C_Receptacle_USB2.0_16P, J2 jst sh 6 pin, J3 Conn_01x04, SW1 SW_SPDT, U1 USBLC6-2SC6, U2 STM32F405RGTx, U3 LM2596S-3.3, U4 SN65HVD232, Y1 16MHz

Commit message: added buzzer, xt30, leds
Parts:
- added BZ1: Buzzer, symbol Device:Buzzer
- added C14: 220u, symbol Device:C
- added C15: 680u, symbol Device:C
- added D4: 1N5822, Diode_THT:D_DO-201AD_P15.24mm_Horizontal, symbol Diode:1N5822
- added D5, D6: LED, symbol Device:LED
- added H1, H2, H3, H4: ~, symbol Mechanical:MountingHole_Pad
- added J4: XT30, symbol Connector_Generic:Conn_01x02
- added L2: 22u, symbol Device:L
- added Q1, Q2: NPN, symbol Simulation_SPICE:NPN
- added R10, R8: 330R, symbol Device:R_Small
- added R11, R9: 56R, symbol Device:R_Small
- added R6: 10k, symbol Device:R
- added R7: 2k2, symbol Device:R
- added U5: LM2596S-5, Package_TO_SOT_SMD:TO-263-5_TabPin3, symbol Regulator_Switching:LM2596S-5
- C12: value 100u -> 330u
Connections:
- net GND: now also BZ1.2 (-), C14.2, C15.2, D4.2 (A), H1.1, H2.1, H3.1, H4.1, J4.1 (Pin_1), Q1.3 (E), Q2.3 (E), R7.2, U5.3 (GND), U5.5 (~{ON}/OFF)
- net VCC: now also C15.1, J4.2 (Pin_2), R10.1, R6.1, R8.1, U5.1 (VIN)
- net PWM_BUZZER: now reaches U2.14 (PA0)
- net PWM_BUZZER: now also BZ1.1 (+)
- net LED1_CTRL: now reaches U2.26 (PB0)
- net LED1_CTRL: now also R9.1
- net LED2_CTRL: now reaches U2.27 (PB1)
- net LED2_CTRL: now also R11.1
- net VBAT_SENSE: now reaches U2.8 (PC0)
- net VBAT_SENSE: now also R6.2, R7.1
- new net: D5.1 (K), R8.2
- new net: D5.2 (A), Q1.1 (C)
- new net: Q1.2 (B), R9.2
- new net: D6.1 (K), R10.2
- new net: D6.2 (A), Q2.1 (C)
- new net: D4.1 (K), L2.1, U5.2 (OUT)
- new net: Q2.2 (B), R11.2
- new net +5V: C14.1, L2.2, U5.4 (FB)
Other:
- note added: "BUZZER"
- note added: "Need higher current buck"
- moved on the sheet: C11, C12, D2, L1, U3

Commit message: added sensors, switch, mounting hole, servo...
Parts:
- removed C1, C2, C3, C4: 100n, symbol Device:C
- removed C14: 220u, symbol Device:C
- removed C15: 680u, symbol Device:C
- removed C5: 10u, symbol Device:C
- removed C6: 10n, symbol Device:C
- removed C7, C8: 1u, symbol Device:C
- removed D3: D_Small, symbol Device:D_Small
- removed D4: 1N5822, Diode_THT:D_DO-201AD_P15.24mm_Horizontal, symbol Diode:1N5822
- removed FB1: 120R, symbol Device:FerriteBead
- removed H1, H2, H3, H4: ~, symbol Mechanical:MountingHole_Pad
- removed J2: jst sh 6 pin, symbol Connector_Generic:Conn_01x06
- removed J3: Conn_01x04, symbol Connector_Generic:Conn_01x04
- removed L2: 22u, symbol Device:L
- removed R2: 10k, symbol Device:R
- removed SW1: SW_SPDT, symbol Switch:SW_SPDT
- removed U5: LM2596S-5, Package_TO_SOT_SMD:TO-263-5_TabPin3, symbol Regulator_Switching:LM2596S-5
- added C14, C15, C16, C19, C20, C26, C27, C28, C29: 100n, symbol Device:C_Small
- added C17, C18, C25: 10u, symbol Device:C_Small
- added C21: 22n, symbol Device:C_Small
- added C22, C23: 15u, symbol Device:C_Small
- added C24: 100p, symbol Device:C_Small
- added C30: 10n, symbol Device:C_Small
- added C31, C32: 1u, symbol Device:C_Small
- added D4: D_Small, symbol Device:D_Small
- added F1: 6A, symbol Device:Polyfuse
- added F2: 1.5A, symbol Device:Polyfuse
- added FB2: 120R, symbol Device:FerriteBead_Small
- added H1, H2, H3, H4: MountingHole, MountingHole:MountingHole_3.2mm_M3, symbol Mechanical:MountingHole
- added J10: servo_3, symbol Connector:Conn_01x03_Pin
- added J11: servo_4, symbol Connector:Conn_01x03_Pin
- added J2: jst gh 4 pin, symbol Connector_Generic_MountingPin:Conn_01x04_MountingPin
- added J3, J6, J7: jst_gh 4 pin, symbol Connector_Generic_MountingPin:Conn_01x04_MountingPin
- added J5: jst sh 6 pin, symbol Connector_Generic_MountingPin:Conn_01x06_MountingPin
- added J8: servo_1, symbol Connector:Conn_01x03_Pin
- added J9: servo_2, symbol Connector:Conn_01x03_Pin
- added L3: 4.7u, symbol Device:L
- added R12: 52.3k, symbol Device:R_Small
- added R15: 90.9k, symbol Device:R_Small
- added R16, R19, R2, R23, R24: 10k, symbol Device:R_Small
- added R17, R20: 5k1, symbol Device:R_Small
- added R18: 50k, symbol Device:R_Small
- added R21: 3k3, symbol Device:R_Small
- added R22: 3k9, symbol Device:R_Small
- added SW1, SW3: SW_Push, symbol Switch:SW_Push
- added SW2: SW_SPST, symbol Switch:SW_SPST
- added U5: ICM-20948, Sensor_Motion:InvenSense_QFN-24_3x3mm_P0.4mm, symbol Sensor_Motion:ICM-20948
- added U6: TPS56A37RPAR, :VQFN-HR-10_L3.0-W3.0_TI_RPA, symbol ACS_easyeda2kicad:TPS56A37RPAR
- added U7: MS5611-01BA, Package_LGA:LGA-8_3x5mm_P1.25mm, symbol Sensor_Pressure:MS5611-01BA
Connections:
- net +3.3V: now also C14.1, C19.1, C25.1, C26.1, C27.1, C28.1, C29.1, C32.1, FB2.2, J3.1 (Pin_1), J5.1 (Pin_1), J6.1 (Pin_1), J7.1 (Pin_1), R17.1, R20.1, R21.1, R23.1, R24.1, SW1.2, U5.13 (VDD), U7.1 (VDD)
- net +3.3VA: now also C30.1, C31.1, FB2.1
- net BOOT0: now also U2.60 (BOOT0), J5.5 (Pin_5)
- net CAN_H: now also J2.2 (Pin_2)
- net CAN_L: now also J2.3 (Pin_3)
- net GND: now also C14.2, C15.2, C16.2, C17.2, C18.2, C19.2, C21.2, C22.2, C23.2, C25.2, C26.2, C27.2, C28.2, C29.2, C30.2, C31.2, C32.2, J10.3 (Pin_3), J11.3 (Pin_3), J2.4 (Pin_4), J2.MP (MountPin), J3.4 (Pin_4), J3.MP (MountPin), J5.2 (Pin_2), J5.MP (MountPin), J6.4 (Pin_4), J6.MP (MountPin), J7.4 (Pin_4), J7.MP (MountPin), J8.3 (Pin_3), J9.3 (Pin_3), R12.2, R16.1, R18.2, R2.1, R22.2, SW2.2 (B), SW3.2, U5.18 (GND), U5.20 (GND), U6.3 (AGND), U6.9 (PGND), U7.2 (PS), U7.3 (GND)
- net NRST: now also J5.6 (Pin_6)
- net PWM_BUZZER: now also U2.23 (PA7); no longer U2.14 (PA0)
- net SWCLK: now also J5.3 (Pin_3)
- net SWDIO: now also J5.4 (Pin_4)
- net VCC: now also D1.1 (K), C16.1, C17.1, D4.1 (K), F1.1, F2.1, U6.8 (VIN); no longer C11.1
- net SWITCH_SENSE: now reaches U2.10 (PC2)
- net SWITCH_SENSE: now also R24.2, SW2.1 (A)
- net PWM_SERVO_2: now reaches U2.15 (PA1)
- net PWM_SERVO_2: now also J9.1 (Pin_1)
- net PWM_SERVO_3: now reaches U2.16 (PA2)
- net PWM_SERVO_3: now also J10.1 (Pin_1)
- net NSS_1: now reaches U2.20 (PA4)
- net NSS_1: now also U7.4 (CSB), U7.5 (CSB)
- net PWM_SERVO_4: now reaches U2.22 (PA6)
- net PWM_SERVO_4: now also J11.1 (Pin_1)
- net EXT_SCL: now reaches U2.29 (PB10)
- net EXT_SCL: now also J6.2 (Pin_2), J7.2 (Pin_2), R17.2, R20.2
- net EXT_SDA: now reaches U2.30 (PB11)
- net EXT_SDA: now also J6.3 (Pin_3), J7.3 (Pin_3)
- net NSS_2: now reaches U2.33 (PB12)
- net NSS_2: now also U5.22 (~{CS})
- net SCK: now reaches U2.34 (PB13)
- net SCK: now also U5.23 (SCL/SCLK), U7.8 (SCLK)
- net MISO: now reaches U2.35 (PB14)
- net MISO: now also U5.9 (SDO/AD0), U7.6 (SDO)
- net MOSI: now reaches U2.36 (PB15)
- net MOSI: now also U5.24 (SDA/SDI), U7.7 (SDI/SDA)
- net UART_TX: now reaches U2.42 (PA9)
- net UART_TX: now also J3.2 (Pin_2)
- net UART_RX: now reaches U2.43 (PA10)
- net UART_RX: now also J3.3 (Pin_3)
- net SCL: now reaches U2.58 (PB6)
- net SDA: now reaches U2.59 (PB7)
- net BUTTON_SENSE: now reaches U2.9 (PC1)
- net BUTTON_SENSE: now also R2.2, R23.2, SW1.1, SW3.1
- new net: C11.1, F2.2
- new net: C15.1, U5.10 (REGOUT)
- new net: D4.2 (A), J2.1 (Pin_1)
- new net: C18.1, F1.2
- new net +6V: C22.1, C23.1, C24.1, J10.2 (Pin_2), J11.2 (Pin_2), J8.2 (Pin_2), J9.2 (Pin_2), L3.2, R15.2, R19.1
- new net BUCK_BOOT: C20.1, U6.7 (BOOT)
- new net BUCK_SW: C20.2, L3.1, U6.6 (SW)
- new net FB: C24.2, R15.1, R16.2, U6.2 (FB)
- new net MODE: R12.1, U6.10 (MODE)
- new net PG: R18.1, R19.2, U6.4 (PG)
- new net PWM_SERVO_1: J8.1 (Pin_1), U2.14 (PA0)
- new net SS: C21.1, U6.5 (SS)
- new net VDDIO: R21.2, R22.1, U5.8 (VDDIO)
- no-connect marks 3 -> 7
Other:
- note added: "LED"
- note added: "OSCILLATOR"
- note added: "POWER MANAGEMENT 3.3V"
- note added: "POWER MANAGEMENT 6V"
- note added: "SENSORS"
- note added: "SERVO"
- note added: "UART/I2C/I2C"
- note added: "USER INPUT"
- note removed: "!!!"
- note removed: "Need higher current buck"
- note removed: "POWER MANAGEMENT"
- moved on the sheet: BZ1, C10, C11, C12, C9, D1, D2, D5, D6, J1, J4, L1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

Commit message: selected LCSC components, small fixes.
Parts:
- removed BZ1: Buzzer, symbol Device:Buzzer
- removed C11: 680u, symbol Device:C
- removed C12: 330u, symbol Device:C
- removed C30: 10n, symbol Device:C_Small
- removed C31, C32: 1u, symbol Device:C_Small
- removed D1, D4: D_Small, symbol Device:D_Small
- removed D2: 1N5822, Diode_THT:D_DO-201AD_P15.24mm_Horizontal, symbol Diode:1N5822
- removed D5, D6: LED, symbol Device:LED
- removed F1: 6A, symbol Device:Polyfuse
- removed F2: 1.5A, symbol Device:Polyfuse
- removed FB2: 120R, symbol Device:FerriteBead_Small
- removed J10: servo_3, symbol Connector:Conn_01x03_Pin
- removed J11: servo_4, symbol Connector:Conn_01x03_Pin
- removed J2: jst gh 4 pin, symbol Connector_Generic_MountingPin:Conn_01x04_MountingPin
- removed J3, J6, J7: jst_gh 4 pin, symbol Connector_Generic_MountingPin:Conn_01x04_MountingPin
- removed J4: XT30, symbol Connector_Generic:Conn_01x02
- removed J5: jst sh 6 pin, symbol Connector_Generic_MountingPin:Conn_01x06_MountingPin
- removed J8: servo_1, symbol Connector:Conn_01x03_Pin
- removed J9: servo_2, symbol Connector:Conn_01x03_Pin
- removed L1: 33u, symbol Device:L
- removed L3: 4.7u, symbol Device:L
- removed Q1, Q2: NPN, symbol Simulation_SPICE:NPN
- removed SW1, SW3: SW_Push, symbol Switch:SW_Push
- removed SW2: SW_SPST, symbol Switch:SW_SPST
- removed U3: LM2596S-3.3, Package_TO_SOT_SMD:TO-263-5_TabPin3, symbol Regulator_Switching:LM2596S-3.3
- removed U4: SN65HVD232, Package_SO:SOIC-8_3.9x4.9mm_P1.27mm, symbol Interface_CAN_LIN:SN65HVD232
- added BUZZER1: 80dB, EasyEDA:BUZ-SMD_4P-L7.5-W7.5-BR, symbol EasyEDA:SMD7525-16Ω
- added C1: 330u, EasyEDA:CAP-SMD_BD10.0-L10.3-W10.3-FD, symbol Device:C
- added C2: 680u, EasyEDA:CAP-SMD_BD10.0-L10.3-W10.3-FD-LS11.0_H12.0, symbol Device:C
- added C3: 100n, Capacitor_SMD:C_0603_1608Metric, symbol Device:C_Small
- added CN1: XT30PW-M, EasyEDA:CONN-TH_XT30PW-M, symbol EasyEDA:XT30PW-M
- added CN2: jst sh 6 pin, EasyEDA:CONN-SMD_6P-P1.00_C9900032244, symbol EasyEDA:D100F1L1-2W6P43
- added CN3, CN4, CN5, CN6: JST_GH 4, EasyEDA:CONN-SMD_4P-P1.25_JXTCONN_DMX-4PWB-43, symbol EasyEDA:DMX-4PWB-43
- added D1, D2, D3: 1N5822, EasyEDA:DO-201AD_BD5.3-L9.5-P13.50-D1.4-RD, symbol EasyEDA:1N5822_C915962
- added F1: 6A, EasyEDA:F1812, symbol EasyEDA:1812L350_16GR
- added F2: 1.5A, EasyEDA:F1812, symbol EasyEDA:mSMD075-33V
- added J4: ARM standard debug, EasyEDA:HDR-SMD_10P-P1.27-V-R2-C5-S5.8, symbol Connector:Conn_ARM_JTAG_SWD_10
- added L1: 4.7u, EasyEDA:IND-TH_L16.0-W8.5-P5.00-D0.7, symbol EasyEDA:PDMTAT044125-4R7MLU
- added L2: 33u, EasyEDA:IND-SMD_L6.8-W6.8_SMMS0630, symbol EasyEDA:SMMS0630-330M
- added LED1: LED BLUE, EasyEDA:LED-SMD_L3.2-W1.0-R-RD, symbol EasyEDA:E6C1204QBAC1UDA
- added LED2: LED GREEN, EasyEDA:LED1206-RD_GREEN-SIDE, symbol EasyEDA:E6CC1206VGAC1UDA
- added LED3: LED RED, EasyEDA:LED1206-RD_RED_XL-3216SURC-FB, symbol EasyEDA:XL-3216SURC-FB
- added Q1, Q2, Q3, Q4: NPN, EasyEDA:SOT-23-3_L2.9-W1.3-P1.90-LS2.4-BR, symbol EasyEDA:BC847B,215
- added R13: 1k, Resistor_SMD:R_0603_1608Metric, symbol Device:R
- added R14: 180R, Resistor_SMD:R_0603_1608Metric, symbol Device:R_Small
- added R25: 1k2, Resistor_SMD:R_0603_1608Metric, symbol Device:R_Small
- added R26: 10k, Resistor_SMD:R_0603_1608Metric, symbol Device:R_Small
- added R27: 1k, Resistor_SMD:R_0603_1608Metric, symbol Device:R_Small
- added SW1, SW4: Button, EasyEDA:SW-SMD_4P-L5.2-W5.2-P3.70-LS6.4, symbol EasyEDA:HX5.2X5.2X2.0HSWITCHTACTILESPST-NO0.05A12V
- added U3: SN65HVD232DR, EasyEDA:SOIC-8_L5.0-W4.0-P1.27-LS6.0-BL, symbol EasyEDA:SN65HVD232DR
- added U4: 2.54_conn 12 pin, EasyEDA:HDR-TH_12P-P2.54-V-M-R2-C6-S2.54, symbol EasyEDA:ZX-PZ2.54-2-6PZZ
- added U8: LM2596S-3.3_C19631822, EasyEDA:TO-263-5_L10.2-W9.0-P1.70-TL-LS15.2, symbol EasyEDA:LM2596S-3.3_C19631822
- added U9: Switch, EasyEDA:SW-TH_MT-0-102-E001-T000-RS-PJ, symbol EasyEDA:MT-0-102-E001-T000-RS
- C10, C9: footprint (none) -> Capacitor_SMD:C_0603_1608Metric; LCSC Part (none) -> C1634
- C13: value 0.1u -> 100n; footprint (none) -> Capacitor_SMD:C_0603_1608Metric; LCSC Part (none) -> C14663
- C14, C15, C16, C19, C20, C26, C27, C28, C29: footprint (none) -> Capacitor_SMD:C_0603_1608Metric; LCSC Part (none) -> C14663
- C17, C18: footprint (none) -> Capacitor_SMD:C_0603_1608Metric; LCSC Part (none) -> C19702
- C21: footprint (none) -> Capacitor_SMD:C_0603_1608Metric; LCSC Part (none) -> C21122
- C22, C23: footprint (none) -> Capacitor_SMD:C_0603_1608Metric; LCSC Part (none) -> C445715
- C24: footprint (none) -> Capacitor_SMD:C_0603_1608Metric; LCSC Part (none) -> C14858
- C25: value 10u -> 100n; footprint (none) -> Capacitor_SMD:C_0603_1608Metric; LCSC Part (none) -> C14663
- H1, H2, H3, H4: footprint MountingHole:MountingHole_3.2mm_M3 -> EasyEDA:SMD_BD4.0-D2.5_TH162030CTJ; LCSC Part (none) -> C3020127
- J1: footprint (none) -> EasyEDA:USB-C-SMD_G-SWITCH_GT-USB-7010ASV; LCSC Part (none) -> C2988369
- R1, R16, R19, R2, R23, R24, R6: footprint (none) -> Resistor_SMD:R_0603_1608Metric; LCSC Part (none) -> C98220
- R10, R8: value 330R -> 150R; footprint (none) -> Resistor_SMD:R_0603_1608Metric; LCSC Part (none) -> C2907103
- R11, R9: value 56R -> 1k2; footprint (none) -> Resistor_SMD:R_0603_1608Metric; LCSC Part (none) -> C2906976
- R12: footprint (none) -> Resistor_SMD:R_0603_1608Metric; LCSC Part (none) -> C2998074
- R15: footprint (none) -> Resistor_SMD:R_0603_1608Metric; LCSC Part (none) -> C2930136
- R17, R20, R3, R4: footprint (none) -> Resistor_SMD:R_0603_1608Metric; LCSC Part (none) -> C2907044
- R18: footprint (none) -> Resistor_SMD:R_0603_1608Metric; LCSC Part (none) -> C861451
- R21: footprint (none) -> Resistor_SMD:R_0603_1608Metric; LCSC Part (none) -> C22978
- R22: footprint (none) -> Resistor_SMD:R_0603_1608Metric; LCSC Part (none) -> C2907024
- R5: footprint (none) -> Resistor_SMD:R_0603_1608Metric; LCSC Part (none) -> C22787
- R7: footprint (none) -> Resistor_SMD:R_0603_1608Metric; LCSC Part (none) -> C114662
- U1: footprint Package_TO_SOT_SMD:SOT-23-6 -> EasyEDA:SOT-23-6_L2.9-W1.6-P0.95-LS2.8-BL; LCSC Part (none) -> C7519
- U2: LCSC Part (none) -> C15742
- U6: footprint :VQFN-HR-10_L3.0-W3.0_TI_RPA -> EasyEDA:VQFN-HR-10_L3.0-W3.0_TI_RPA
- U7: footprint Package_LGA:LGA-8_3x5mm_P1.25mm -> EasyEDA:SENSORS-SMD_MS5611-01BA03; LCSC Part (none) -> C15639
- Y1: footprint (none) -> EasyEDA:CRYSTAL-SMD_4P-L3.2-W2.5-BL; LCSC Part (none) -> C112972
Connections:
- net +3.3VA is gone; now on net +3.3V: U2.13 (VDDA)
- net +3.3V: now also BUZZER1.1, C1.1, C3.1, CN2.1, CN4.1, CN5.1, CN6.1, L2.2, SW4.2, U3.3 (VCC), U8.4 (Feedback)
- net +6V: now also R10.1, R8.1, L1.2, R14.1, U4.10, U4.3, U4.4, U4.9
- net BOOT0: now also R2.2, CN2.5, SW4.3
- net BUCK_SW: now also L1.1
- net BUTTON_SENSE: now also SW1.3; no longer R2.2
- net CAN_H: now also CN3.2, U3.7 (CANH)
- net CAN_L: now also CN3.3, U3.6 (CANL)
- net CAN_RX: now also U3.4 (R)
- net CAN_TX: now also U3.1 (D)
- net EXT_SCL: now also CN5.2, CN6.2
- net EXT_SDA: now also CN5.3, CN6.3
- net GND: now also C1.2, C2.2, C3.2, CN1.1 (-), CN1.3, CN1.4, CN2.2, CN2.7, CN2.8, CN3.4, CN3.5, CN3.6, CN4.4, CN4.5, CN4.6, CN5.4, CN5.5, CN5.6, CN6.4, CN6.5, CN6.6, D3.2 (A), J4.3 (GND), J4.5 (GND), J4.9 (GNDDetect), Q1.2, Q2.2, Q3.2, Q4.2, R26.2, SW1.2, U3.2 (GND), U4.11, U4.12, U4.5, U4.6, U8.3 (Gnd), U8.5 (~{ON}/OFF), U8.6 (TAB), U9.3
- net NRST: now also CN2.6, J4.10 (~{RESET})
- net PWM_BUZZER: now also R26.1, R27.1
- net PWM_SERVO_1: now also U4.1
- net PWM_SERVO_2: now also U4.2
- net PWM_SERVO_3: now also U4.7
- net PWM_SERVO_4: now also U4.8
- net SWCLK: now also CN2.3, J4.4 (SWCLK/TCK)
- net SWDIO: now also CN2.4, J4.2 (SWDIO/TMS)
- net SWITCH_SENSE: now also U9.2
- net UART_RX: now also CN4.3
- net UART_TX: now also CN4.2
- net VCC: now also CN1.2 (+), D1.1 (K), D2.1 (K), F1.1, F2.1, U8.1 (Vin); no longer R10.1, R8.1
- net at R8.2: now also LED2.1 (K)
- net at R9.2: now also Q1.1
- net LEDR_CTRL: now reaches U2.28 (PB2)
- net LEDR_CTRL: now also R25.1
- net at R10.2: now also LED1.2 (-)
- net at R11.2: now also Q3.1
- net at J1.A4 (VBUS), J1.A9 (VBUS), J1.B4 (VBUS)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: now also D2.2 (A)
- net at C18.1: now also F1.2
- net LED1_CTRL renamed LEDG_CTRL
- net LED2_CTRL renamed LEDB_CTRL
- net SCL: no longer names the net of U2.58 (PB6)
- net SDA: no longer names the net of U2.59 (PB7)
- new net: LED3.1 (K), R14.2
- new net: BUZZER1.2, Q4.3
- new net: Q2.1, R25.2
- new net: LED3.2 (A), Q2.3
- new net: J4.1 (VTref), R13.2
- new net: LED2.2 (A), Q1.3
- new net: LED1.1 (+), Q3.3
- new net: Q4.1, R27.2
- new net: CN3.1, D1.2 (A)
- new net: C2.1, F2.2
- new net +3V3: R13.1
- new net OUTPUT: D3.1 (K), L2.1, U8.2 (Output)
- no-connect marks 7 -> 45
Other:
- note added: "DO NOT PLACE COPPER DIRECTLY BELOW"
- note added: "V_f = 2.3V, I = 20mA"
- note added: "V_f = 3.0V, I = 20mA"
- moved on the sheet: C13, C25, C26, C27, C28, C29, H1, R1, R10, R11, R24, R5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

Commit message: fixed things noted in design review
Parts:
- removed C2: 680u, EasyEDA:CAP-SMD_BD10.0-L10.3-W10.3-FD-LS11.0_H12.0, symbol Device:C
- removed D1, D2, D3: 1N5822, EasyEDA:DO-201AD_BD5.3-L9.5-P13.50-D1.4-RD, symbol EasyEDA:1N5822_C915962
- removed R21: 3k3, Resistor_SMD:R_0603_1608Metric, symbol Device:R_Small
- removed R22: 3k9, Resistor_SMD:R_0603_1608Metric, symbol Device:R_Small
- added C11, C12, C8: 22u, Capacitor_SMD:C_0603_1608Metric, symbol Device:C_Small
- added C4, C6: 1u, Capacitor_SMD:C_0603_1608Metric, symbol Device:C_Small
- added C5, C7: 10u, Capacitor_SMD:C_0201_0603Metric, symbol Device:C
- added D1, D2, D3, D4, D5, D6, D7: SS34, EasyEDA:SMC_L6.9-W5.9-LS7.9-RD, symbol EasyEDA:SS34_C154551
- added F3: 1.5A, EasyEDA:F1812, symbol EasyEDA:mSMD075-33V
- added U10: ME6206B18XG, EasyEDA:SOT-23-3_L2.9-W1.3-P1.90-LS2.4-BR, symbol EasyEDA:ME6206B18XG
- C1: value 330u -> 10u; footprint EasyEDA:CAP-SMD_BD10.0-L10.3-W10.3-FD -> Capacitor_SMD:C_0201_0603Metric; LCSC Part C250072 -> C19702
Connections:
- net +3.3V: now also C5.1, C6.1, C7.1, D5.2 (A), D6.2 (A), D7.2 (A), U10.3 (VIN); no longer CN4.1, CN5.1, CN6.1
- net GND: now also C11.2, C12.2, C4.2, C5.2, C6.2, C7.2, C8.2, D3.2 (A), U10.1 (VSS)
- net OUTPUT: now also F2.2, U8.1 (Vin), C11.1, C12.1, C8.1, D3.1 (C), F3.2
- net VBUS: now also D2.1 (C), D4.2 (A)
- net VCC: now also D1.1 (C); no longer C16.1, C17.1, U6.8 (VIN), U8.1 (Vin)
- net VDDIO: now also C4.1, U10.2 (VOUT)
- net at R14.2: now also LED3.2 (A); no longer LED3.1 (K)
- net at C18.1, F1.2: now also C16.1, C17.1, U6.8 (VIN)
- net at Q2.3: now also LED3.1 (K); no longer LED3.2 (A)
- net at Q1.3: now also LED2.1 (K); no longer LED2.2 (A)
- net at R10.2: now also LED1.1 (+); no longer LED1.2 (-)
- net at Q3.3: now also LED1.2 (-); no longer LED1.1 (+)
- net at CN3.1: now also D1.2 (A)
- net at J1.A4 (VBUS), J1.A9 (VBUS), J1.B4 (VBUS)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: now also D2.2 (A)
- net at R8.2: now also LED2.2 (A); no longer LED2.1 (K)
- new net: CN4.1, D6.1 (C)
- new net: CN5.1, D5.1 (C)
- new net: D4.1 (C), F3.1
- new net: CN6.1, D7.1 (C)
Other:
- moved on the sheet: C14, C15, C19, CN1, CN4, CN5, CN6, F1, F2, LED1, LED2, LED3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

Commit message: placement stuff
Parts:
- removed CN1: XT30PW-M, EasyEDA:CONN-TH_XT30PW-M, symbol EasyEDA:XT30PW-M
- removed D2: SS34, EasyEDA:SMC_L6.9-W5.9-LS7.9-RD, symbol EasyEDA:SS34_C154551
- removed J1: USB_C_Receptacle_USB2.0_16P, EasyEDA:USB-C-SMD_G-SWITCH_GT-USB-7010ASV, symbol Connector:USB_C_Receptacle_USB2.0_16P
- removed L1: 4.7u, EasyEDA:IND-TH_L16.0-W8.5-P5.00-D0.7, symbol EasyEDA:PDMTAT044125-4R7MLU
- removed R3, R4: 5k1, Resistor_SMD:R_0603_1608Metric, symbol Device:R
- added CN_BAT1: XT30, EasyEDA:CONN-TH_XT30UPB-M, symbol EasyEDA:XT30UPB-M
- added D8: SS34, EasyEDA:SMC_L6.9-W5.9-LS7.9-RD, symbol EasyEDA:SS34_C154551
- added J2: GT-USB-7010ASV, EasyEDA:USB-C-SMD_G-SWITCH_GT-USB-7010ASV, symbol EasyEDA:GT-USB-7010ASV
- added L3: 4.7u, EasyEDA:L0603, symbol EasyEDA:LQM18PN4R7MFRL
- added R22, R28: 5k1, Resistor_SMD:R_0603_1608Metric, symbol Device:R
- renumbered CN3 to CN_CAN1, CN5 to CN_I2C_1, CN6 to CN_I2C_2, CN4 to CN_UART1, SW4 to SW_BOOT0, SW1 to SW_BUTTON1, U9 to U_SWITCH1
Connections:
- net +6V: now also L3.2
- net BUCK_SW: now also L3.1
- net GND: now also CN_BAT1.1 (-), J2.1 (SHELL), J2.2 (SHELL), J2.3 (SHELL), J2.4 (SHELL), J2.A1B12 (GND), J2.B1A12 (GND), R22.2, R28.1
- net OUTPUT: no longer C11.1, C12.1, C8.1, F2.2, F3.2, U8.1 (Vin)
- net USB_ESD+: now also J2.A6 (DP1), J2.B6 (DP2)
- net USB_ESD-: now also J2.A7 (DN1), J2.B7 (DN2)
- net VBUS: now also D8.1 (C)
- net VCC: now also CN_BAT1.2 (+)
- new net: D8.2 (A), J2.A4B9 (VBUS), J2.B4A9 (VBUS)
- new net: J2.A5 (CC1), R22.1
- new net: J2.B5 (CC2), R28.2
- new net: C11.1, C12.1, C8.1, F2.2, F3.2, U8.1 (Vin)
Other:
- note removed: "AN4879*"

Commit message: finished layout
Parts:
- removed CN2: jst sh 6 pin, EasyEDA:CONN-SMD_6P-P1.00_C9900032244, symbol EasyEDA:D100F1L1-2W6P43
- removed CN_I2C_1, CN_I2C_2, CN_UART1: JST_GH 4, EasyEDA:CONN-SMD_4P-P1.25_JXTCONN_DMX-4PWB-43, symbol EasyEDA:DMX-4PWB-43
- removed D5, D6, D7: SS34, EasyEDA:SMC_L6.9-W5.9-LS7.9-RD, symbol EasyEDA:SS34_C154551
- removed R17, R20: 5k1, Resistor_SMD:R_0603_1608Metric, symbol Device:R_Small
- removed R23: 10k, Resistor_SMD:R_0603_1608Metric, symbol Device:R_Small
- removed SW_BUTTON1: Button, EasyEDA:SW-SMD_4P-L5.2-W5.2-P3.70-LS6.4, symbol EasyEDA:HX5.2X5.2X2.0HSWITCHTACTILESPST-NO0.05A12V
- added H5: MountingHole_Pad, MountingHole:MountingHole_2.2mm_M2_DIN965_Pad, symbol Mechanical:MountingHole_Pad
Connections:
- net +3V3 is gone; now on net +3.3V: R13.1
- net GND: now also H5.1
- net BUTTON_SENSE: no longer names the net of U2.9 (PC1)
- net EXT_SCL: no longer names the net of U2.29 (PB10)
- net EXT_SDA: no longer names the net of U2.30 (PB11)
- net UART_RX: no longer names the net of U2.43 (PA10)
- net UART_TX: no longer names the net of U2.42 (PA9)
- no-connect marks 45 -> 49
Other:
- note removed: "UART/I2C/I2C"
- moved on the sheet: C10, C9, J4, LED1, LED2, LED3, Q1, Q2, Q3, R10, R11, R13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
